File: hardware/ttc_sign_v2/ttc_sign_v2.kicad_sch (KiCad schematic)
At the start: 37 parts, among them J1 USB_B_Mini, J2 PROG, Q1 2N7002, Q2 2N7002, Q3 2N7002, Q4 2N7002, Q5 S8050, Q6 S8050, SW1 SW_Push, SW2 SW_Push, SW3 SW_Push, SW4 SW_Push, U1 DISPLAY, U2 CD40109, U3 74HC595, U4 ESP32-WROOM-32D, U5 AP1117-33

Commit message: Moved and uploaded hardware files
Parts:
- removed Q5, Q6: S8050, Package_TO_SOT_SMD:SOT-23, symbol Device:Q_NPN_BEC
- removed R2: 10k, Resistor_SMD:R_0603_1608Metric, symbol Device:R_US
- added D1, D2: LED, LED_SMD:LED_0805_2012Metric, symbol Device:LED
- added R1, R4: 330, Resistor_SMD:R_0603_1608Metric, symbol Device:R_US
- added R5, R6, R7: 10k, Resistor_SMD:R_0603_1608Metric, symbol Device:R_US
- U1: renamed from U4; footprint RF_Module:ESP32-WROOM-32 -> RF_Module:ESP32-WROOM-32D
- renumbered C4 to C1, C3 to C10, C7 to C2, C1 to C3, C8 to C4, C2 to C5, C9 to C6, C10 to C7, C5 to C8, C6 to C9, R1 to R2, U5 to U3, U3 to U4, U1 to U5
Connections:
- net +3V3 is gone; now on net +3.3V: C3.1, C5.2, C9.1, R2.2, U1.2 (VDD), U2.1 (VLOW), U2.15 (END), U2.2 (ENA), U2.7 (ENB), U2.9 (ENC), U3.2 (VO)
- net DTR is gone; now on net +3.3V: J2.2 (Pin_2)
- net BOOT: now also J2.6 (Pin_6)
- net BUT_{1}: now also R3.2
- net BUT_{2}: now also R5.2
- net EN: now also J2.1 (Pin_1)
- net GND: now also J2.4 (Pin_4), D1.1 (K), D2.1 (K); no longer J2.1 (Pin_1)
- net RX: now also J2.5 (Pin_5); no longer J2.6 (Pin_6)
- net SW_{3}: now also R6.2
- net SW_{4}: now also R7.2
- net TX: now also J2.3 (Pin_3); no longer J2.4 (Pin_4)
- net LED_{1}: now reaches U1.12 (IO27)
- net LED_{1}: now also R1.1
- net LED_{2}: now reaches U1.9 (IO33)
- net LED_{2}: now also R4.1
- net +3.3V: now reaches R3.1
- net +3.3V: now also R5.1, R6.1, R7.1
- removed net RTS: J2.3 (Pin_3), R3.2
- new net: D2.2 (A), R4.2
- new net: D1.2 (A), R1.2
- no-connect marks 22 -> 19
Other:
- note added: "Buttons should need at least 100g force to press"
- note added: "Make surface mount"
- note added: "Move to USB-C or Micro-USB"
- note added: "Programming interfaces and hardware to enable UART programming with ESP-PROG"
- note removed: "Programming interfaces and hardware to enable UART programming"
- note removed: "RTS = CTS"
- moved on the sheet: C4, C6, C7, JP1, JP2, SW2, SW3, SW4
